File: boneIO - relay board 32x10A.kicad_pcb (KiCad board)
At the start: 2 copper layers, 197 x 102 mm, 241 parts, among them J1 Screw_Terminal_01x03, J10 Screw_Terminal_01x03, J11 Screw_Terminal_01x03, J12 Conn_02x04_Odd_Even, J13 Screw_Terminal_01x03, J14 Screw_Terminal_01x03, J15 Screw_Terminal_01x03, J16 Screw_Terminal_01x03, J17 Screw_Terminal_01x03, J2 Screw_Terminal_01x03, J3 Screw_Terminal_01x03, J4 Screw_Terminal_01x03, J5 Screw_Terminal_01x03, J6 Screw_Terminal_01x03, J7 Screw_Terminal_01x03, J8 Screw_Terminal_01x03, J9 Screw_Terminal_01x03, K1 HF32F/024-ZS3, K10 HF32F/024-ZS3, K11 HF32F/024-ZS3, K12 HF32F/024-ZS3, K13 HF32F/024-ZS3, K14 HF32F/024-ZS3, K15 HF32F/024-ZS3, K16 HF32F/024-ZS3, K17 HF32F/024-ZS3, K18 HF32F/024-ZS3, K19 HF32F/024-ZS3, K2 HF32F/024-ZS3, K20 HF32F/024-ZS3, K21 HF32F/024-ZS3, K22 HF32F/024-ZS3, K23 HF32F/024-ZS3, K24 HF32F/024-ZS3, K25 HF32F/024-ZS3, K26 HF32F/024-ZS3, K27 HF32F/024-ZS3, K28 HF32F/024-ZS3, K29 HF32F/024-ZS3, K3 HF32F/024-ZS3, K30 HF32F/024-ZS3, K31 HF32F/024-ZS3, K32 HF32F/024-ZS3, K4 HF32F/024-ZS3, K5 HF32F/024-ZS3, K6 HF32F/024-ZS3, K7 HF32F/024-ZS3, K8 HF32F/024-ZS3, K9 HF32F/024-ZS3, Q1 BC817, Q10 BC817, Q11 BC817, Q12 BC817, Q13 BC817, Q14 BC817, Q15 BC817, Q16 BC817, Q17 BC817, Q18 BC817, Q19 BC817, Q2 BC817, Q20 BC817, Q21 BC817, Q22 BC817, Q23 BC817, Q24 BC817, Q25 BC817, Q26 BC817, Q27 BC817, Q28 BC817, Q29 BC817, Q3 BC817, Q30 BC817, Q31 BC817, Q32 BC817, Q4 BC817, Q5 BC817, Q6 BC817, Q7 BC817, Q8 BC817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

Commit message: v0.4
Parts:
- removed SW1, SW2, SW3: SW_DIP_x03, Button_Switch_SMD:SW_DIP_SPSTx03_Slide_Omron_A6S-310x_W8.9mm_P2.54mm
- added JP10: SolderJumper_2_Open, Jumper:SolderJumper-2_P1.3mm_Open_RoundedPad1.0x1.5mm, F.Cu at (482.2, 308.2)
- added JP11: SolderJumper_3_Bridged12, Jumper:SolderJumper-3_P1.3mm_Bridged2Bar12_RoundedPad1.0x1.5mm, B.Cu at (379.4, 317.2)
- added JP2: SolderJumper_2_Open, Jumper:SolderJumper-2_P1.3mm_Open_RoundedPad1.0x1.5mm, F.Cu at (369.4, 311.7)
- added JP3: SolderJumper_2_Open, Jumper:SolderJumper-2_P1.3mm_Open_RoundedPad1.0x1.5mm, F.Cu at (366.9, 311.7)
- added JP4: SolderJumper_2_Bridged, Jumper:SolderJumper-2_P1.3mm_Bridged_RoundedPad1.0x1.5mm, F.Cu at (364.4, 311.7)
- added JP5: SolderJumper_2_Open, Jumper:SolderJumper-2_P1.3mm_Open_RoundedPad1.0x1.5mm, F.Cu at (399.8, 311.7)
- added JP6: SolderJumper_2_Open, Jumper:SolderJumper-2_P1.3mm_Open_RoundedPad1.0x1.5mm, F.Cu at (397.3, 311.7)
- added JP7: SolderJumper_2_Open, Jumper:SolderJumper-2_P1.3mm_Open_RoundedPad1.0x1.5mm, F.Cu at (394.8, 311.7)
- added JP8: SolderJumper_2_Open, Jumper:SolderJumper-2_P1.3mm_Open_RoundedPad1.0x1.5mm, F.Cu at (477.1, 308.2)
- added JP9: SolderJumper_2_Open, Jumper:SolderJumper-2_P1.3mm_Open_RoundedPad1.0x1.5mm, F.Cu at (479.6, 308.2)
- added K33: HF49FD/005-1H12T, HF49FD_005-1H12T (1):RELAY_HF49FD_005-1H11T, F.Cu at (297.9, 337.7)
- added K34: HF49FD/005-1H12T, HF49FD_005-1H12T (1):RELAY_HF49FD_005-1H11T, F.Cu at (309.1, 337.6)
- added K35: HF49FD/005-1H12T, HF49FD_005-1H12T (1):RELAY_HF49FD_005-1H11T, F.Cu at (333.5, 337.7)
- added K36: HF49FD/005-1H12T, HF49FD_005-1H12T (1):RELAY_HF49FD_005-1H11T, F.Cu at (322.3, 337.7)
- added K37: HF49FD/005-1H12T, HF49FD_005-1H12T (1):RELAY_HF49FD_005-1H11T, F.Cu at (346.6, 337.7)
- added K38: HF49FD/005-1H12T, HF49FD_005-1H12T (1):RELAY_HF49FD_005-1H11T, F.Cu at (357.8, 337.7)
- added K39: HF49FD/005-1H12T, HF49FD_005-1H12T (1):RELAY_HF49FD_005-1H11T, F.Cu at (370.9, 337.7)
- added K40: HF49FD/005-1H12T, HF49FD_005-1H12T (1):RELAY_HF49FD_005-1H11T, F.Cu at (382.1, 337.7)
- added K41: HF49FD/005-1H12T, HF49FD_005-1H12T (1):RELAY_HF49FD_005-1H11T, F.Cu at (406.4, 337.7)
- added K42: HF49FD/005-1H12T, HF49FD_005-1H12T (1):RELAY_HF49FD_005-1H11T, F.Cu at (395.2, 337.7)
- added K43: HF49FD/005-1H12T, HF49FD_005-1H12T (1):RELAY_HF49FD_005-1H11T, F.Cu at (430.8, 337.7)
- added K44: HF49FD/005-1H12T, HF49FD_005-1H12T (1):RELAY_HF49FD_005-1H11T, F.Cu at (419.6, 337.7)
- added K45: HF49FD/005-1H12T, HF49FD_005-1H12T (1):RELAY_HF49FD_005-1H11T, F.Cu at (443.9, 337.6)
- added K46: HF49FD/005-1H12T, HF49FD_005-1H12T (1):RELAY_HF49FD_005-1H11T, F.Cu at (455.1, 337.6)
- added K47: HF49FD/005-1H12T, HF49FD_005-1H12T (1):RELAY_HF49FD_005-1H11T, F.Cu at (468.2, 337.7)
- added K48: HF49FD/005-1H12T, HF49FD_005-1H12T (1):RELAY_HF49FD_005-1H11T, F.Cu at (479.4, 337.7)
- added K49: HF49FD/005-1H12T, HF49FD_005-1H12T (1):RELAY_HF49FD_005-1H11T, F.Cu at (304.9, 285.9)
- added K50: HF49FD/005-1H12T, HF49FD_005-1H12T (1):RELAY_HF49FD_005-1H11T, F.Cu at (293.7, 285.9)
- added K51: HF49FD/005-1H12T, HF49FD_005-1H12T (1):RELAY_HF49FD_005-1H11T, F.Cu at (329.2, 285.9)
- added K52: HF49FD/005-1H12T, HF49FD_005-1H12T (1):RELAY_HF49FD_005-1H11T, F.Cu at (318.0, 285.9)
- added K53: HF49FD/005-1H12T, HF49FD_005-1H12T (1):RELAY_HF49FD_005-1H11T, F.Cu at (353.5, 285.9)
- added K54: HF49FD/005-1H12T, HF49FD_005-1H12T (1):RELAY_HF49FD_005-1H11T, F.Cu at (342.3, 285.9)
- added K55: HF49FD/005-1H12T, HF49FD_005-1H12T (1):RELAY_HF49FD_005-1H11T, F.Cu at (426.5, 285.9)
- added K56: HF49FD/005-1H12T, HF49FD_005-1H12T (1):RELAY_HF49FD_005-1H11T, F.Cu at (415.3, 285.9)
- added K57: HF49FD/005-1H12T, HF49FD_005-1H12T (1):RELAY_HF49FD_005-1H11T, F.Cu at (402.1, 285.9)
- added K58: HF49FD/005-1H12T, HF49FD_005-1H12T (1):RELAY_HF49FD_005-1H11T, F.Cu at (391.0, 285.9)
- added K59: HF49FD/005-1H12T, HF49FD_005-1H12T (1):RELAY_HF49FD_005-1H11T, F.Cu at (377.9, 285.9)
- added K60: HF49FD/005-1H12T, HF49FD_005-1H12T (1):RELAY_HF49FD_005-1H11T, F.Cu at (366.6, 285.9)
- added K61: HF49FD/005-1H12T, HF49FD_005-1H12T (1):RELAY_HF49FD_005-1H11T, F.Cu at (450.9, 285.9)
- added K62: HF49FD/005-1H12T, HF49FD_005-1H12T (1):RELAY_HF49FD_005-1H11T, F.Cu at (439.6, 285.9)
- added K63: HF49FD/005-1H12T, HF49FD_005-1H12T (1):RELAY_HF49FD_005-1H11T, F.Cu at (475.2, 285.9)
- added K64: HF49FD/005-1H12T, HF49FD_005-1H12T (1):RELAY_HF49FD_005-1H11T, F.Cu at (463.9, 285.9)
- added Q10: BC817, Package_TO_SOT_SMD:SOT-23, B.Cu at (334.9, 325.3)
- added Q11: BC817, Package_TO_SOT_SMD:SOT-23, B.Cu at (347.9, 325.3)
- added Q12: BC817, Package_TO_SOT_SMD:SOT-23, B.Cu at (358.6, 325.2)
- added Q19: BC817, Package_TO_SOT_SMD:SOT-23, B.Cu at (372.3, 325.3)
- added Q20: BC817, Package_TO_SOT_SMD:SOT-23, B.Cu at (383.5, 325.2)
- added Q21: BC817, Package_TO_SOT_SMD:SOT-23, B.Cu at (396.6, 325.2)
- added Q22: BC817, Package_TO_SOT_SMD:SOT-23, B.Cu at (407.8, 325.2)
- added Q23: BC817, Package_TO_SOT_SMD:SOT-23, B.Cu at (421.0, 325.2)
- added Q24: BC817, Package_TO_SOT_SMD:SOT-23, B.Cu at (432.2, 325.2)
- added Q25: BC817, Package_TO_SOT_SMD:SOT-23, B.Cu at (303.5, 298.3)
- added Q26: BC817, Package_TO_SOT_SMD:SOT-23, B.Cu at (292.8, 298.3)
- added Q27: BC817, Package_TO_SOT_SMD:SOT-23, B.Cu at (327.8, 298.3)
- added Q28: BC817, Package_TO_SOT_SMD:SOT-23, B.Cu at (316.7, 298.3)
- added Q29: BC817, Package_TO_SOT_SMD:SOT-23, B.Cu at (352.2, 298.3)
- added Q30: BC817, Package_TO_SOT_SMD:SOT-23, B.Cu at (341.0, 298.3)
- added Q37: BC817, Package_TO_SOT_SMD:SOT-23, B.Cu at (376.6, 298.3)
- added Q38: BC817, Package_TO_SOT_SMD:SOT-23, B.Cu at (365.3, 298.3)
- added Q39: BC817, Package_TO_SOT_SMD:SOT-23, B.Cu at (400.8, 298.3)
- added Q40: BC817, Package_TO_SOT_SMD:SOT-23, B.Cu at (389.6, 298.3)
- added Q41: BC817, Package_TO_SOT_SMD:SOT-23, B.Cu at (425.2, 298.3)
- added Q42: BC817, Package_TO_SOT_SMD:SOT-23, B.Cu at (414.4, 298.3)
- added Q49: BC817, Package_TO_SOT_SMD:SOT-23, B.Cu at (449.5, 298.3)
- added Q50: BC817, Package_TO_SOT_SMD:SOT-23, B.Cu at (438.3, 298.3)
- added Q51: BC817, Package_TO_SOT_SMD:SOT-23, B.Cu at (473.8, 298.3)
- added Q52: BC817, Package_TO_SOT_SMD:SOT-23, B.Cu at (462.6, 298.3)
- added Q61: BC817, Package_TO_SOT_SMD:SOT-23, B.Cu at (445.3, 325.2)
- added Q62: BC817, Package_TO_SOT_SMD:SOT-23, B.Cu at (456.4, 325.2)
- added Q63: BC817, Package_TO_SOT_SMD:SOT-23, B.Cu at (469.6, 325.2)
- added Q64: BC817, Package_TO_SOT_SMD:SOT-23, B.Cu at (480.8, 325.2)
- added Q7: BC817, Package_TO_SOT_SMD:SOT-23, B.Cu at (299.0, 325.3)
- added Q8: BC817, Package_TO_SOT_SMD:SOT-23, B.Cu at (310.1, 325.3)
- added Q9: BC817, Package_TO_SOT_SMD:SOT-23, B.Cu at (323.7, 325.3)
- added R103: 4.7k, Resistor_SMD:R_0603_1608Metric, B.Cu at (448.7, 325.1)
- added R104: 4.7k, Resistor_SMD:R_0603_1608Metric, B.Cu at (459.8, 325.1)
- added R105: 4.7k, Resistor_SMD:R_0603_1608Metric, B.Cu at (472.8, 325.1)
- added R106: 4.7k, Resistor_SMD:R_0603_1608Metric, B.Cu at (483.9, 325.1)
- added R13: 4.7k, Resistor_SMD:R_0603_1608Metric, B.Cu at (362.2, 325.2)
- added R29: 4.7k, Resistor_SMD:R_0603_1608Metric, B.Cu at (375.5, 325.2)
- added R30: 4.7k, Resistor_SMD:R_0603_1608Metric, B.Cu at (386.7, 325.2)
- added R31: 4.7k, Resistor_SMD:R_0603_1608Metric, B.Cu at (400.0, 325.1)
- added R32: 4.7k, Resistor_SMD:R_0603_1608Metric, B.Cu at (411.0, 325.1)
- added R33: 4.7k, Resistor_SMD:R_0603_1608Metric, B.Cu at (424.3, 325.1)
- added R34: 4.7k, Resistor_SMD:R_0603_1608Metric, B.Cu at (435.6, 325.1)
- added R47: 4.7k, Resistor_SMD:R_0603_1608Metric, B.Cu at (300.4, 298.4)
- added R48: 4.7k, Resistor_SMD:R_0603_1608Metric, B.Cu at (290.1, 298.4)
- added R49: 4.7k, Resistor_SMD:R_0603_1608Metric, B.Cu at (324.7, 298.4)
- added R50: 4.7k, Resistor_SMD:R_0603_1608Metric, B.Cu at (313.4, 298.4)
- added R51: 4.7k, Resistor_SMD:R_0603_1608Metric, B.Cu at (348.9, 298.4)
- added R52: 4.7k, Resistor_SMD:R_0603_1608Metric, B.Cu at (337.8, 298.4)
- added R69: 4.7k, Resistor_SMD:R_0603_1608Metric, B.Cu at (373.3, 298.4)
- added R70: 4.7k, Resistor_SMD:R_0603_1608Metric, B.Cu at (362.0, 298.4)
- added R71: 4.7k, Resistor_SMD:R_0603_1608Metric, B.Cu at (397.7, 298.4)
- added R72: 4.7k, Resistor_SMD:R_0603_1608Metric, B.Cu at (386.6, 298.4)
- added R73: 4.7k, Resistor_SMD:R_0603_1608Metric, B.Cu at (422.0, 298.4)
- added R74: 4.7k, Resistor_SMD:R_0603_1608Metric, B.Cu at (410.8, 298.4)
- added R8: 4.7k, Resistor_SMD:R_0603_1608Metric, B.Cu at (302.1, 325.1)
- added R82: 10k, Resistor_SMD:R_0603_1608Metric, F.Cu at (477.1, 311.7)
- added R83: 10k, Resistor_SMD:R_0603_1608Metric, F.Cu at (479.7, 311.7)
- added R84: 10k, Resistor_SMD:R_0603_1608Metric, F.Cu at (482.2, 311.7)
- added R9: 4.7k, Resistor_SMD:R_0603_1608Metric, B.Cu at (313.2, 325.1)
- added R91: 4.7k, Resistor_SMD:R_0603_1608Metric, B.Cu at (446.4, 298.4)
- added R92: 4.7k, Resistor_SMD:R_0603_1608Metric, B.Cu at (434.9, 298.4)
- added R93: 4.7k, Resistor_SMD:R_0603_1608Metric, B.Cu at (470.7, 298.4)
- added R94: 4.7k, Resistor_SMD:R_0603_1608Metric, B.Cu at (459.3, 298.4)
- added REF**: OSHW-Logo2_14.6x12mm_SilkScreen, Symbol:OSHW-Logo2_14.6x12mm_SilkScreen, F.Cu at (450.3, 312.1)
- R10, R11, R12: value 10k -> 4.7k; moved to B.Cu
- moved R10 143.1 mm to (326.9, 325.1), turned to -90 degrees
- moved R11 131.7 mm to (338.1, 325.1), turned to -90 degrees
- moved R12 118.4 mm to (351.2, 325.1), turned to -90 degrees
- moved R62 11.6 mm to (394.8, 315.2), turned to -90 degrees
- moved R14 11.2 mm to (369.4, 315.2), turned to -90 degrees
- moved R61 8.65 mm to (397.3, 315.2), turned to -90 degrees
- moved R21 8.25 mm to (366.8, 315.2), turned to -90 degrees
- moved C7 8.22 mm to (471.4, 308.9)
- moved R86 8.22 mm to (471.3, 307.1)
- moved R85 8.22 mm to (471.3, 305.2)
- moved R60 6.05 mm to (399.8, 315.2), turned to -90 degrees
- moved U29 5.99 mm to (471.1, 313.9)
- moved U30 5.99 mm to (471.1, 313.9)
- moved R22 5.88 mm to (364.4, 315.2), turned to -90 degrees
- moved JP1 2.61 mm to (384.5, 317.3)
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- renumbered C2 to C1, C1 to C2, C9 to C7, D17 to D13, D18 to D14, D19 to D15, D20 to D16, D21 to D17, D22 to D18, D23 to D19, D24 to D20, D25 to D21, D26 to D22, D27 to D23, D28 to D24, D29 to D25, D30 to D26, D31 to D27, D32 to D28, D13 to D29, D14 to D30, D15 to D31, D16 to D32, J13 to J10, J14 to J11, J15 to J12, J12 to J13, J7 to J14, J8 to J15, J9 to J7, J10 to J8, J11 to J9, K17 to K13, K18 to K14, K19 to K15, K20 to K16, K21 to K17, K22 to K18, K23 to K19, K24 to K20, K25 to K21, K26 to K22, K27 to K23, K28 to K24, K29 to K25, K30 to K26, K31 to K27, K32 to K28, K13 to K29, K14 to K30, K15 to K31, K16 to K32, Q7 to Q13, Q8 to Q14, Q17 to Q15, Q18 to Q16, Q19 to Q17, Q20 to Q18, Q10 to Q31, Q9 to Q32, Q11 to Q33, Q12 to Q34, Q13 to Q35, Q14 to Q36, Q15 to Q43, Q16 to Q44, Q26 to Q45, Q25 to Q46, Q27 to Q47, Q28 to Q48, Q29 to Q53, Q30 to Q54, Q31 to Q55, Q32 to Q56, Q21 to Q57, Q22 to Q58, Q23 to Q59, Q24 to Q60, R59 to R100, R60 to R101, R57 to R102, R56 to R107, R58 to R108, R61 to R109, R62 to R110, R2 to R14, R21 to R15, R17 to R16, R19 to R17, R24 to R18, R25 to R19, R15 to R2, R26 to R20, R3 to R21, R4 to R22, R27 to R23, R28 to R24, R47 to R25, R49 to R26, R51 to R27, R52 to R28, R16 to R3, R29 to R35, R30 to R36, R48 to R37, R50 to R38, R53 to R39, R18 to R4, R54 to R40, R33 to R41, R31 to R42, R35 to R43, R36 to R44, R39 to R45, R40 to R46, R20 to R5, R5 to R53, R34 to R54, R32 to R55, R37 to R56, R38 to R57, R41 to R58, R42 to R59, R22 to R6, R6 to R60, R7 to R61, R8 to R62, R43 to R63, R44 to R64, R63 to R66, R23 to R7, R45 to R75, R46 to R76, R66 to R77, R64 to R78, R69 to R79, R70 to R80, R9 to R81, R13 to R85, R14 to R86, R71 to R87, R72 to R88, R75 to R89, R76 to R90, R73 to R95, R74 to R96, R77 to R97, R78 to R98, R55 to R99, U15 to U10, U24 to U11, U26 to U12, U27 to U13, U28 to U14, U5 to U15, U17 to U16, U16 to U17, U7 to U22, U22 to U23, U23 to U24, U34 to U25, U33 to U26, U35 to U27, U36 to U28, U9 to U29, U4 to U3, U10 to U30, U37 to U31, U38 to U32, U39 to U33, U40 to U34, U29 to U35, U30 to U36, U31 to U37, U32 to U38, U6 to U4, U8 to U5, U12 to U6, U13 to U7, U3 to U8, U14 to U9
Connections:
- net Net-(D1-Pad2) renamed P0_1_OUT
- net Net-(D10-Pad2) renamed P9_1_OUT
- net Net-(D11-Pad2) renamed P10_1_OUT
- net Net-(D12-Pad2) renamed P11_1_OUT
- net Net-(D13-Pad2) renamed P12_1_OUT
- net Net-(D14-Pad2) renamed P13_1_OUT
- net Net-(D15-Pad2) renamed P14_1_OUT
- net Net-(D16-Pad2) renamed P15_1_OUT
- net Net-(D17-Pad2) renamed P17_1_OUT
- net Net-(D18-Pad2) renamed P16_1_OUT
- net Net-(D19-Pad2) renamed P19_1_OUT
- net Net-(D2-Pad2) renamed P1_1_OUT
- net Net-(D20-Pad2) renamed P18_1_OUT
- net Net-(D21-Pad2) renamed P21_1_OUT
- net Net-(D22-Pad2) renamed P20_1_OUT
- net Net-(D23-Pad2) renamed P23_1_OUT
- net Net-(D24-Pad2) renamed P22_1_OUT
- net Net-(D25-Pad2) renamed P25_1_OUT
- net Net-(D26-Pad2) renamed P24_1_OUT
- net Net-(D27-Pad2) renamed P27_1_OUT
- net Net-(D28-Pad2) renamed P26_1_OUT
- net Net-(D29-Pad2) renamed P29_1_OUT
- net Net-(D3-Pad2) renamed P2_1_OUT
- net Net-(D30-Pad2) renamed P28_1_OUT
- net Net-(D31-Pad2) renamed P31_1_OUT
- net Net-(D32-Pad2) renamed P30_1_OUT
- net Net-(D4-Pad2) renamed P3_1_OUT
- net Net-(D5-Pad2) renamed P4_1_OUT
- net Net-(D6-Pad2) renamed P5_1_OUT
- net Net-(D7-Pad2) renamed P6_1_OUT
- net Net-(D8-Pad2) renamed P7_1_OUT
- net Net-(D9-Pad2) renamed P8_1_OUT
- net Net-(R22-Pad2) renamed /R5
- net Net-(R27-Pad2) renamed /R7
- net Net-(R28-Pad2) renamed /R8
- net Net-(R32-Pad2) renamed /R14
- net Net-(R34-Pad2) renamed /R13
- net Net-(R47-Pad2) renamed /R9
- net Net-(R49-Pad2) renamed /R10
- net Net-(R51-Pad2) renamed /R11
- net Net-(R52-Pad2) renamed /R12
- net Net-(R55-Pad2) renamed /R29
- net Net-(R57-Pad2) renamed /R30
- net Net-(R59-Pad2) renamed /R31
- net Net-(R60-Pad2) renamed /R32
- net Net-(R69-Pad2) renamed /R23
- net Net-(R70-Pad2) renamed /R24
- net Net-(R73-Pad2) renamed /R25
- net Net-(R74-Pad2) renamed /R26
- net Net-(R77-Pad2) renamed /R27
- net Net-(R78-Pad2) renamed /R28
- J13 pad 1: VCC -> +24V
- R10 pad 1: Net-(R10-Pad1) -> Net-(Q9-Pad1)
- R10 pad 2: GND -> /R4
- R11 pad 1: Net-(R11-Pad1) -> Net-(Q10-Pad1)
- R11 pad 2: GND -> /R3
- R12 pad 1: Net-(R12-Pad1) -> Net-(Q11-Pad1)
- R12 pad 2: GND -> /R6
- R2 pad 2: Net-(R15-Pad2) (its old number) -> /R1
- R3 pad 2: Net-(R16-Pad2) (its old number) -> /R2
- R4 pad 2: Net-(R18-Pad2) (its old number) -> /R3
- R5 pad 2: Net-(R20-Pad2) (its old number) -> /R4
- R56 pad 2: Net-(R37-Pad2) (its old number) -> /R15
- R57 pad 2: Net-(R38-Pad2) (its old number) -> /R16
- R58 pad 2: Net-(R41-Pad2) (its old number) -> /R17
- R59 pad 2: Net-(R42-Pad2) (its old number) -> /R18
- R7 pad 2: Net-(R23-Pad2) -> /R6
- R75 pad 2: Net-(R45-Pad2) (its old number) -> /R19
- R76 pad 2: Net-(R46-Pad2) (its old number) -> /R20
- R77 pad 2: Net-(R66-Pad2) (its old number) -> /R21
- R78 pad 2: Net-(R64-Pad2) (its old number) -> /R22
- U18 pad 3: Net-(R37-Pad2) (its old number) -> /R15
- U19 pad 3: Net-(R38-Pad2) (its old number) -> /R16
- U2 pad 3: Net-(R15-Pad2) (its old number) -> /R1
- U20 pad 3: Net-(R41-Pad2) (its old number) -> /R17
- U21 pad 3: Net-(R42-Pad2) (its old number) -> /R18
- U23 pad 3: Net-(R45-Pad2) (its old number) -> /R19
- U24 pad 3: Net-(R46-Pad2) (its old number) -> /R20
- U25 pad 3: Net-(R66-Pad2) (its old number) -> /R21
- U26 pad 3: Net-(R64-Pad2) (its old number) -> /R22
- U29 pad 5: Net-(R12-Pad1) -> Net-(JP10-Pad2)
- U29 pad 6: Net-(R11-Pad1) -> Net-(JP9-Pad2)
- U29 pad 7: Net-(R10-Pad1) -> Net-(JP8-Pad2)
- U3 pad 3: Net-(R16-Pad2) (its old number) -> /R2
- U30 pad 5: Net-(R12-Pad1) -> Net-(JP10-Pad2)
- U30 pad 6: Net-(R11-Pad1) -> Net-(JP9-Pad2)
- U30 pad 7: Net-(R10-Pad1) -> Net-(JP8-Pad2)
- U4 pad 3: Net-(R18-Pad2) (its old number) -> /R3
- U5 pad 3: Net-(R20-Pad2) (its old number) -> /R4
- U7 pad 3: Net-(R23-Pad2) -> /R6
Routing:
- net VCC: track 879.3 -> 931.7 mm, vias 32 -> 30
- net Net-(R12-Pad1): track 36.0 -> 0.00 mm, vias 4 -> 0
- net Net-(R11-Pad1): track 35.4 -> 0.00 mm, vias 4 -> 0
- net Net-(R10-Pad1): track 33.2 -> 0.00 mm, vias 2 -> 0
- net /R19: track 0.00 -> 33.2 mm, vias 0 -> 1
- net Net-(J8-Pad1): track 56.8 -> 89.7 mm
- net Net-(J17-Pad1): track 56.8 -> 89.7 mm
- net Net-(J10-Pad1): track 56.8 -> 89.7 mm
- net Net-(J11-Pad1): track 56.8 -> 89.7 mm
- net Net-(J16-Pad1): track 56.8 -> 89.7 mm
- net Net-(J7-Pad1): track 56.8 -> 89.7 mm
- net Net-(J9-Pad1): track 56.8 -> 89.7 mm
- net Net-(J12-Pad1): track 56.8 -> 89.7 mm
- net /R3: track 0.00 -> 32.9 mm, vias 0 -> 1
- net /R17: track 0.00 -> 32.5 mm, vias 0 -> 1
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Other:
- outline, holes or cut-outs redrawn
- board text added: "+24V"
- board text added: "+5V"
- board text added: "0x20"
- board text added: "0x21"
- board text added: "0x48"
- board text added: "CONTROL EXPANDER"
- board text added: "CONTROL RELAY"
- board text added: "address"
- board text added: "relay board 32x10A v0.4.0 MIX"
- board text removed: "Temp Sensor"
- board text removed: "relay board 32x10A v0.2"
