File: boneIO - relay board 32x10A.kicad_sch (KiCad schematic)
At the start: 240 parts, among them J1 Screw_Terminal_01x03, J10 Screw_Terminal_01x03, J11 Screw_Terminal_01x03, J12 Conn_02x04_Odd_Even, J13 Screw_Terminal_01x03, J14 Screw_Terminal_01x03, J15 Screw_Terminal_01x03, J16 Screw_Terminal_01x03, J17 Screw_Terminal_01x03, J2 Screw_Terminal_01x03, J3 Screw_Terminal_01x03, J4 Screw_Terminal_01x03, J5 Screw_Terminal_01x03, J6 Screw_Terminal_01x03, J7 Screw_Terminal_01x03, J8 Screw_Terminal_01x03, J9 Screw_Terminal_01x03, K1 HF32F/024-ZS3, K10 HF32F/024-ZS3, K11 HF32F/024-ZS3, K12 HF32F/024-ZS3, K13 HF32F/024-ZS3, K14 HF32F/024-ZS3, K15 HF32F/024-ZS3, K16 HF32F/024-ZS3, K17 HF32F/024-ZS3, K18 HF32F/024-ZS3, K19 HF32F/024-ZS3, K2 HF32F/024-ZS3, K20 HF32F/024-ZS3, K21 HF32F/024-ZS3, K22 HF32F/024-ZS3, K23 HF32F/024-ZS3, K24 HF32F/024-ZS3, K25 HF32F/024-ZS3, K26 HF32F/024-ZS3, K27 HF32F/024-ZS3, K28 HF32F/024-ZS3, K29 HF32F/024-ZS3, K3 HF32F/024-ZS3, K30 HF32F/024-ZS3, K31 HF32F/024-ZS3, K32 HF32F/024-ZS3, K4 HF32F/024-ZS3, K5 HF32F/024-ZS3, K6 HF32F/024-ZS3, K7 HF32F/024-ZS3, K8 HF32F/024-ZS3, K9 HF32F/024-ZS3, Q1 BC817, Q10 BC817, Q11 BC817, Q12 BC817, Q13 BC817, Q14 BC817, Q15 BC817, Q16 BC817, Q17 BC817, Q18 BC817, Q19 BC817, Q2 BC817, Q20 BC817, Q21 BC817, Q22 BC817, Q23 BC817, Q24 BC817, Q25 BC817, Q26 BC817, Q27 BC817, Q28 BC817, Q29 BC817, Q3 BC817, Q30 BC817, Q31 BC817, Q32 BC817, Q4 BC817, Q5 BC817, Q6 BC817, Q7 BC817, Q8 BC817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

Commit message: v0.4
Parts:
- removed SW1, SW2, SW3: SW_DIP_x03, Button_Switch_SMD:SW_DIP_SPSTx03_Slide_Omron_A6S-310x_W8.9mm_P2.54mm, symbol Switch:SW_DIP_x03
- added JP10, JP2, JP3, JP5, JP6, JP7, JP8, JP9: SolderJumper_2_Open, Jumper:SolderJumper-2_P1.3mm_Open_RoundedPad1.0x1.5mm, symbol Jumper:SolderJumper_2_Open
- added JP11: SolderJumper_3_Bridged12, Jumper:SolderJumper-3_P1.3mm_Bridged2Bar12_RoundedPad1.0x1.5mm, symbol Jumper:SolderJumper_3_Bridged12
- added JP4: SolderJumper_2_Bridged, Jumper:SolderJumper-2_P1.3mm_Bridged_RoundedPad1.0x1.5mm, symbol Jumper:SolderJumper_2_Bridged
- added K33, K34, K35, K36, K37, K38, K39, K40, K41, K42, K43, K44, K45, K46, K47, K48, K49, K50, K51, K52, K53, K54, K55, K56, K57, K58, K59, K60, K61, K62, K63, K64: HF49FD/005-1H12T, HF49FD_005-1H12T (1):RELAY_HF49FD_005-1H11T, symbol HF49FD_005-1H12T:HF49FD/005-1H12T
- added Q10, Q11, Q12, Q19, Q20, Q21, Q22, Q23, Q24, Q25, Q26, Q27, Q28, Q29, Q30, Q37, Q38, Q39, Q40, Q41, Q42, Q49, Q50, Q51, Q52, Q61, Q62, Q63, Q64, Q7, Q8, Q9: BC817, Package_TO_SOT_SMD:SOT-23, symbol Transistor_BJT:BC817
- added R103, R104, R105, R106, R13, R29, R30, R31, R32, R33, R34, R47, R48, R49, R50, R51, R52, R69, R70, R71, R72, R73, R74, R8, R9, R91, R92, R93, R94: 4.7k, Resistor_SMD:R_0603_1608Metric, symbol Device:R
- added R82, R83, R84: 10k, Resistor_SMD:R_0603_1608Metric, symbol Device:R
- R10, R11, R12: value 10k -> 4.7k
- renumbered C2 to C1, C1 to C2, C9 to C7, D17 to D13, D18 to D14, D19 to D15, D20 to D16, D21 to D17, D22 to D18, D23 to D19, D24 to D20, D25 to D21, D26 to D22, D27 to D23, D28 to D24, D29 to D25, D30 to D26, D31 to D27, D32 to D28, D13 to D29, D14 to D30, D15 to D31, D16 to D32, J13 to J10, J14 to J11, J15 to J12, J12 to J13, J7 to J14, J8 to J15, J9 to J7, J10 to J8, J11 to J9, K17 to K13, K18 to K14, K19 to K15, K20 to K16, K21 to K17, K22 to K18, K23 to K19, K24 to K20, K25 to K21, K26 to K22, K27 to K23, K28 to K24, K29 to K25, K30 to K26, K31 to K27, K32 to K28, K13 to K29, K14 to K30, K15 to K31, K16 to K32, Q7 to Q13, Q8 to Q14, Q17 to Q15, Q18 to Q16, Q19 to Q17, Q20 to Q18, Q10 to Q31, Q9 to Q32, Q11 to Q33, Q12 to Q34, Q13 to Q35, Q14 to Q36, Q15 to Q43, Q16 to Q44, Q26 to Q45, Q25 to Q46, Q27 to Q47, Q28 to Q48, Q29 to Q53, Q30 to Q54, Q31 to Q55, Q32 to Q56, Q21 to Q57, Q22 to Q58, Q23 to Q59, Q24 to Q60, R59 to R100, R60 to R101, R57 to R102, R56 to R107, R58 to R108, R61 to R109, R62 to R110, R2 to R14, R21 to R15, R17 to R16, R19 to R17, R24 to R18, R25 to R19, R15 to R2, R26 to R20, R3 to R21, R4 to R22, R27 to R23, R28 to R24, R47 to R25, R49 to R26, R51 to R27, R52 to R28, R16 to R3, R29 to R35, R30 to R36, R48 to R37, R50 to R38, R53 to R39, R18 to R4, R54 to R40, R33 to R41, R31 to R42, R35 to R43, R36 to R44, R39 to R45, R40 to R46, R20 to R5, R5 to R53, R34 to R54, R32 to R55, R37 to R56, R38 to R57, R41 to R58, R42 to R59, R22 to R6, R6 to R60, R7 to R61, R8 to R62, R43 to R63, R44 to R64, R63 to R66, R23 to R7, R45 to R75, R46 to R76, R66 to R77, R64 to R78, R69 to R79, R70 to R80, R9 to R81, R13 to R85, R14 to R86, R71 to R87, R72 to R88, R75 to R89, R76 to R90, R73 to R95, R74 to R96, R77 to R97, R78 to R98, R55 to R99, U15 to U10, U24 to U11, U26 to U12, U27 to U13, U28 to U14, U5 to U15, U17 to U16, U16 to U17, U7 to U22, U22 to U23, U23 to U24, U34 to U25, U33 to U26, U35 to U27, U36 to U28, U9 to U29, U4 to U3, U10 to U30, U37 to U31, U38 to U32, U39 to U33, U40 to U34, U29 to U35, U30 to U36, U31 to U37, U32 to U38, U6 to U4, U8 to U5, U12 to U6, U13 to U7, U3 to U8, U14 to U9
Connections:
- net +24V: now also J13.1 (Pin_1), JP11.1 (A)
- net +3V3: now also JP10.1 (A), JP2.1 (A), JP3.1 (A), JP4.1 (A), JP5.1 (A), JP6.1 (A), JP7.1 (A), JP8.1 (A), JP9.1 (A)
- net +5V: now also JP11.3 (B)
- net A0_1: now also JP4.2 (B)
- net A0_2: now also JP7.2 (B)
- net A1_1: now also JP3.2 (B)
- net A1_2: now also JP6.2 (B)
- net A2_1: now also JP2.2 (B)
- net A2_2: now also JP5.2 (B)
- net GND: now also R82.2, R83.2, R84.2; no longer R10.2, R11.2, R12.2
- net GND1: now also Q10.2 (E), Q11.2 (E), Q12.2 (E), Q19.2 (E), Q20.2 (E), Q21.2 (E), Q22.2 (E), Q23.2 (E), Q24.2 (E), Q25.2 (E), Q26.2 (E), Q27.2 (E), Q28.2 (E), Q29.2 (E), Q30.2 (E), Q37.2 (E), Q38.2 (E), Q39.2 (E), Q40.2 (E), Q41.2 (E), Q42.2 (E), Q49.2 (E), Q50.2 (E), Q51.2 (E), Q52.2 (E), Q61.2 (E), Q62.2 (E), Q63.2 (E), Q64.2 (E), Q7.2 (E), Q8.2 (E), Q9.2 (E)
- net VCC: now also JP11.2 (C), K33.2, K34.2, K35.2, K36.2, K37.2, K38.2, K39.2, K40.2, K41.2, K42.2, K43.2, K44.2, K45.2, K46.2, K47.2, K48.2, K49.2, K50.2, K51.2, K52.2, K53.2, K54.2, K55.2, K56.2, K57.2, K58.2, K59.2, K60.2, K61.2, K62.2, K63.2, K64.2; no longer J13.1 (Pin_1)
- net at U29.5 (A2), U30.5 (A2): now also JP10.2 (B), R84.1; no longer R12.1
- net at U29.6 (A1), U30.6 (A1): now also JP9.2 (B), R83.1; no longer R11.1
- net at U29.7 (A0), U30.7 (A0): now also JP8.2 (B), R82.1; no longer R10.1
- net at J1.1 (Pin_1), K1.4, K2.4: now also K33.3, K34.3
- net at J1.2 (Pin_2), K1.3: now also K33.4
- net at J1.3 (Pin_3), K2.3: now also K34.4
- net at J2.1 (Pin_1), K3.4, K4.4: now also K35.3, K36.3
- net at J2.2 (Pin_2), K3.3: now also K36.4
- net at J2.3 (Pin_3), K4.3: now also K35.4
- net at J3.1 (Pin_1), K5.4, K6.4: now also K37.3, K38.3
- net at J3.2 (Pin_2), K5.3: now also K37.4
- net at J3.3 (Pin_3), K6.3: now also K38.4
- net at J4.1 (Pin_1), K7.4, K8.4: now also K39.3, K40.3
- net at J4.2 (Pin_2), K7.3: now also K39.4
- net at J4.3 (Pin_3), K8.3: now also K40.4
- net at J5.1 (Pin_1), K10.4, K9.4: now also K41.3, K42.3
- net at J5.2 (Pin_2), K9.3: now also K42.4
- net at J5.3 (Pin_3), K10.3: now also K41.4
- net at J6.1 (Pin_1), K11.4, K12.4: now also K43.3, K44.3
- net at J6.2 (Pin_2), K11.3: now also K44.4
- net at J6.3 (Pin_3), K12.3: now also K43.4
- net at J14.1 (Pin_1), K29.4, K30.4: now also K45.3, K46.3
- net at J14.2 (Pin_2), K29.3: now also K45.4
- net at J14.3 (Pin_3), K30.3: now also K46.4
- net at J15.1 (Pin_1), K31.4, K32.4: now also K47.3, K48.3
- net at J15.2 (Pin_2), K31.3: now also K47.4
- net at J15.3 (Pin_3), K32.3: now also K48.4
- net at J7.1 (Pin_1), K13.4, K14.4: now also K49.3, K50.3
- net at J7.2 (Pin_2), K13.3: now also K49.4
- net at J7.3 (Pin_3), K14.3: now also K50.4
- net at J8.1 (Pin_1), K15.4, K16.4: now also K51.3, K52.3
- net at J8.2 (Pin_2), K15.3: now also K51.4
- net at J8.3 (Pin_3), K16.3: now also K52.4
- net at J9.1 (Pin_1), K17.4, K18.4: now also K53.3, K54.3
- net at J9.2 (Pin_2), K17.3: now also K53.4
- net at J9.3 (Pin_3), K18.3: now also K54.4
- net at J10.1 (Pin_1), K19.4, K20.4: now also K59.3, K60.3
- net at J10.2 (Pin_2), K19.3: now also K59.4
- net at J10.3 (Pin_3), K20.3: now also K60.4
- net at J11.1 (Pin_1), K21.4, K22.4: now also K57.3, K58.3
- net at J11.2 (Pin_2), K21.3: now also K57.4
- net at J11.3 (Pin_3), K22.3: now also K58.4
- net at J12.1 (Pin_1), K23.4, K24.4: now also K55.3, K56.3
- net at J12.2 (Pin_2), K23.3: now also K55.4
- net at J12.3 (Pin_3), K24.3: now also K56.4
- net at J16.1 (Pin_1), K25.4, K26.4: now also K61.3, K62.3
- net at J16.2 (Pin_2), K25.3: now also K61.4
- net at J16.3 (Pin_3), K26.3: now also K62.4
- net at J17.1 (Pin_1), K27.4, K28.4: now also K63.3, K64.3
- net at J17.2 (Pin_2), K27.3: now also K63.4
- net at J17.3 (Pin_3), K28.3: now also K64.4
- net at Q56.1 (B), R98.1: now also Q52.3 (C)
- net R28: now reaches R98.2, U34.3
- net R28: now also R93.2
- net at Q3.1 (B), R4.1: now also Q9.3 (C)
- net P2_1_OUT: now reaches D3.2 (A), K3.5, Q3.3 (C)
- net P2_1_OUT: now also K36.1
- net P9_1_OUT: now reaches D10.2 (A), K10.5, Q16.3 (C)
- net P9_1_OUT: now also K41.1
- net P15_1_OUT: now reaches D32.2 (A), K32.5, Q60.3 (C)
- net P15_1_OUT: now also K48.1
- net at Q2.1 (B), R3.1: now also Q8.3 (C)
- net P1_1_OUT: now reaches D2.2 (A), K2.5, Q2.3 (C)
- net P1_1_OUT: now also K34.1
- net at Q44.1 (B), R76.1: now also Q38.3 (C)
- net P22_1_OUT: now reaches D20.2 (A), K20.5, Q44.3 (C)
- net P22_1_OUT: now also K60.1
- net P27_1_OUT: now reaches D23.2 (A), K23.5, Q47.3 (C)
- net P27_1_OUT: now also K55.1
- net P5_1_OUT: now reaches D6.2 (A), K6.5, Q6.3 (C)
- net P5_1_OUT: now also K38.1
- net at Q47.1 (B), R79.1: now also Q41.3 (C)
- net R23: now reaches R79.2, U27.3
- net R23: now also R74.2
- net P24_1_OUT: now reaches D22.2 (A), K22.5, Q46.3 (C)
- net P24_1_OUT: now also K58.1
- net P20_1_OUT: now reaches D18.2 (A), K18.5, Q36.3 (C)
- net P20_1_OUT: now also K54.1
- net P3_1_OUT: now reaches D4.2 (A), K4.5, Q4.3 (C)
- net P3_1_OUT: now also K35.1
- net R25: now reaches R95.2, U31.3
- net R25: now also R92.2
- net R11: now reaches R27.2, U13.3
- net R11: now also R34.2
- net at Q33.1 (B), R56.1: now also Q27.3 (C)
- net R15: now reaches R56.2, U18.3
- net R15: now also R50.2
- net at Q36.1 (B), R59.1: now also Q30.3 (C)
- net R18: now reaches R59.2, U21.3
- net R18: now also R51.2
- net at Q59.1 (B), R100.1: now also Q63.3 (C)
- net R31: now reaches R100.2, U37.3
- net R31: now also R106.2
- net P31_1_OUT: now reaches D27.2 (A), K27.5, Q55.3 (C)
- net P31_1_OUT: now also K63.1
- net P30_1_OUT: now reaches D28.2 (A), K28.5, Q56.3 (C)
- net P30_1_OUT: now also K64.1
- net R30: now reaches R102.2, U36.3
- net R30: now also R103.2
- net at Q14.1 (B), R24.1: now also Q20.3 (C)
- net R8: now reaches R24.2, U10.3
- net R8: now also R29.2
- net P28_1_OUT: now reaches D26.2 (A), K26.5, Q54.3 (C)
- net P28_1_OUT: now also K62.1
- net at Q35.1 (B), R58.1: now also Q29.3 (C)
- net R17: now reaches R58.2, U20.3
- net R17: now also R52.2
- net R10: now reaches R26.2, U12.3
- net R10: now also R31.2
- net at Q48.1 (B), R80.1: now also Q42.3 (C)
- net P26_1_OUT: now reaches D24.2 (A), K24.5, Q48.3 (C)
- net P26_1_OUT: now also K56.1
- net P12_1_OUT: now reaches D29.2 (A), K29.5, Q57.3 (C)
- net P12_1_OUT: now also K45.1
- net at Q55.1 (B), R97.1: now also Q51.3 (C)
- net at Q15.1 (B), R25.1: now also Q21.3 (C)
- net P8_1_OUT: now reaches D9.2 (A), K9.5, Q15.3 (C)
- net P8_1_OUT: now also K42.1
- net P19_1_OUT: now reaches D15.2 (A), K15.5, Q33.3 (C)
- net P19_1_OUT: now also K51.1
- net P6_1_OUT: now reaches D7.2 (A), K7.5, Q13.3 (C)
- net P6_1_OUT: now also K39.1
- net at Q13.1 (B), R23.1: now also Q19.3 (C)
- net P16_1_OUT: now reaches D14.2 (A), K14.5, Q32.3 (C)
- net P16_1_OUT: now also K50.1
- net at Q53.1 (B), R95.1: now also Q49.3 (C)
- net P29_1_OUT: now reaches D25.2 (A), K25.5, Q53.3 (C)
- net P29_1_OUT: now also K61.1
- net at Q18.1 (B), R28.1: now also Q24.3 (C)
- net P11_1_OUT: now reaches D12.2 (A), K12.5, Q18.3 (C)
- net P11_1_OUT: now also K43.1
- net at Q58.1 (B), R102.1: now also Q62.3 (C)
- net at Q16.1 (B), R26.1: now also Q22.3 (C)
- net at Q31.1 (B), R54.1: now also Q25.3 (C)
- net P17_1_OUT: now reaches D13.2 (A), K13.5, Q31.3 (C)
- net P17_1_OUT: now also K49.1
- net P14_1_OUT: now reaches D31.2 (A), K31.5, Q59.3 (C)
- net P14_1_OUT: now also K47.1
- net P13_1_OUT: now reaches D30.2 (A), K30.5, Q58.3 (C)
- net P13_1_OUT: now also K46.1
- net R27: now reaches R97.2, U33.3
- net R27: now also R94.2
- net P4_1_OUT: now reaches D5.2 (A), K5.5, Q5.3 (C)
- net P4_1_OUT: now also K37.1
- net at Q54.1 (B), R96.1: now also Q50.3 (C)
- net at Q32.1 (B), R55.1: now also Q26.3 (C)
- net R29: now reaches R99.2, U35.3
- net R29: now also R104.2
- net at Q17.1 (B), R27.1: now also Q23.3 (C)
- net P10_1_OUT: now reaches D11.2 (A), K11.5, Q17.3 (C)
- net P10_1_OUT: now also K44.1
- net P7_1_OUT: now reaches D8.2 (A), K8.5, Q14.3 (C)
- net P7_1_OUT: now also K40.1
- net P0_1_OUT: now reaches D1.2 (A), K1.5, Q1.3 (C)
- net P0_1_OUT: now also K33.1
- net R24: now reaches R80.2, U28.3
- net R24: now also R73.2
- net P25_1_OUT: now reaches D21.2 (A), K21.5, Q45.3 (C)
- net P25_1_OUT: now also K57.1
- net R4: now reaches R5.2, U5.3
- net R4: now also R10.2
- net R22: now reaches R78.2, U26.3
- net R22: now also R71.2
- net at Q6.1 (B), R7.1: now also Q12.3 (C)
- net R3: now reaches R4.2, U4.3
- net R3: now also R11.2
- net P21_1_OUT: now reaches D17.2 (A), K17.5, Q35.3 (C)
- net P21_1_OUT: now also K53.1
- net P23_1_OUT: now reaches D19.2 (A), K19.5, Q43.3 (C)
- net P23_1_OUT: now also K59.1
- net P18_1_OUT: now reaches D16.2 (A), K16.5, Q34.3 (C)
- net P18_1_OUT: now also K52.1
- net R21: now reaches R77.2, U25.3
- net R21: now also R72.2
- net at Q60.1 (B), R101.1: now also Q64.3 (C)
- net R14: now reaches R55.2, U17.3
- net R14: now also R47.2
- net at Q5.1 (B), R6.1: now also Q11.3 (C)
- net R5: now reaches R6.2, U6.3
- net R5: now also R13.2
- net at Q4.1 (B), R5.1: now also Q10.3 (C)
- net R12: now reaches R28.2, U14.3
- net R12: now also R33.2
- net at Q1.1 (B), R2.1: now also Q7.3 (C)
- net at Q43.1 (B), R75.1: now also Q37.3 (C)
- net R19: now reaches R75.2, U23.3
- net R19: now also R70.2
- net R26: now reaches R96.2, U32.3
- net R26: now also R91.2
- net at Q34.1 (B), R57.1: now also Q28.3 (C)
- net at Q45.1 (B), R77.1: now also Q39.3 (C)
- net R9: now reaches R25.2, U11.3
- net R9: now also R32.2
- net R6: now reaches R7.2, U7.3
- net R6: now also R12.2
- net R20: now reaches R76.2, U24.3
- net R20: now also R69.2
- net at Q57.1 (B), R99.1: now also Q61.3 (C)
- net at Q46.1 (B), R78.1: now also Q40.3 (C)
- net R13: now reaches R54.2, U16.3
- net R13: now also R48.2
- net R1: now reaches R2.2, U2.3
- net R1: now also R9.2
- net R7: now reaches R23.2, U9.3
- net R7: now also R30.2
- net R2: now reaches R3.2, U3.3
- net R2: now also R8.2
- net R32: now reaches R101.2, U38.3
- net R32: now also R105.2
- net R16: now reaches R57.2, U19.3
- net R16: now also R49.2
- new net: Q25.1 (B), R47.1
- new net: Q27.1 (B), R49.1
- new net: Q9.1 (B), R10.1
- new net: Q8.1 (B), R9.1
- new net: Q30.1 (B), R52.1
- new net: Q7.1 (B), R8.1
- new net: Q51.1 (B), R93.1
- new net: Q22.1 (B), R32.1
- new net: Q50.1 (B), R92.1
- new net: Q64.1 (B), R106.1
- new net: Q42.1 (B), R74.1
- new net: Q12.1 (B), R13.1
- new net: Q37.1 (B), R69.1
- new net: Q63.1 (B), R105.1
- new net: Q11.1 (B), R12.1
- new net: Q20.1 (B), R30.1
- new net: Q19.1 (B), R29.1
- new net: Q10.1 (B), R11.1
- new net: Q40.1 (B), R72.1
- new net: Q49.1 (B), R91.1
- new net: Q29.1 (B), R51.1
- new net: Q28.1 (B), R50.1
- new net: Q61.1 (B), R103.1
- new net: Q52.1 (B), R94.1
- new net: Q38.1 (B), R70.1
- new net: Q41.1 (B), R73.1
- new net: Q62.1 (B), R104.1
- new net: Q21.1 (B), R31.1
- new net: Q39.1 (B), R71.1
- new net: Q26.1 (B), R48.1
- new net: Q23.1 (B), R33.1
- new net: Q24.1 (B), R34.1
Other:
- note added: "- relay board 32x10A v4.0"
- note removed: "- relay board 32x10A v1.0"
- moved on the sheet: D1, D10, D11, D12, D13, D14, D15, D16, D17, D18, D19, D2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
